Commit message: backup

File: my_robot/urdf/my_robot.xacro (robot description, xacro)
@@ -9,12 +9,12 @@
   </joint>
   <link name='chassis'>
-    <pose>0 0 0.1 0 0 0</pose>
+    <pose>0 0 -0.1 0 0 0</pose>
     <inertial>
-      <mass value="30.0"/>
-      <origin xyz="0.0 0 0" rpy=" 0 0 0"/>
+      <mass value="20.0"/>
+      <origin xyz="0 0 0" rpy=" 0 0 0"/>
       <inertia
-          ixx="1.975" ixy="0" ixz="0"
-          iyy="1.975" iyz="0"
-          izz="3.75"
+          ixx="0.5" ixy="0" ixz="0"
+          iyy="0.5" iyz="0"
+          izz="0.5"
       />
     </inertial>
@@ -26,5 +26,5 @@
     </collision>
     <visual name='chassis_visual'>
-      <origin xyz="0 0 0" rpy=" 0 0 0"/>
+      <origin xyz="0 0 -0.1" rpy=" 0 0 0"/>
       <geometry>
         <cylinder radius=".5" length=".2"/>
@@ -32,5 +32,5 @@
     </visual>
     <collision name='body_tower'>
-      <origin xyz="0 0 0" rpy=" 0 0 0"/>
+      <origin xyz="0 0 0.3" rpy=" 0 0 0"/>
       <geometry>
         <box size="0.5 0.5 1"/>
@@ -38,5 +38,5 @@
     </collision>
     <visual name='body_tower'>
-      <origin xyz="0 0 0" rpy=" 0 0 0"/>
+      <origin xyz="0 0 0.3" rpy=" 0 0 0"/>
       <geometry>
         <box size="0.5 0.5 1"/>
@@ -44,13 +44,25 @@
     </visual>
     <collision name='back_caster_collision'>
-      <origin xyz="0.45 0 -0.05" rpy=" 0 0 0"/>
+      <origin xyz="0.35 0 -0.22" rpy=" 0 0 0"/>
       <geometry>
-        <sphere radius="0.0499"/>
+        <sphere radius="0.15"/>
       </geometry>
     </collision>
     <visual name='back_caster_visual'>
-      <origin xyz="0.45 0 -0.05" rpy=" 0 0 0"/>
+      <origin xyz="0.35 0 -0.22" rpy=" 0 0 0"/>
       <geometry>
-        <sphere radius="0.05"/>
+        <sphere radius="0.15"/>
+      </geometry>
+    </visual>
+    <collision name='front_caster_collision'>
+      <origin xyz="-0.35 0 -0.22" rpy=" 0 0 0"/>
+      <geometry>
+        <sphere radius="0.15"/>
+      </geometry>
+    </collision>
+    <visual name='front_caster_visual'>
+      <origin xyz="-0.35 0 -0.22" rpy=" 0 0 0"/>
+      <geometry>
+        <sphere radius="0.15"/>
       </geometry>
     </visual>
@@ -61,7 +73,7 @@
       <origin xyz="0 0 0" rpy=" 0 0 0"/>
       <inertia
-          ixx="0.033" ixy="0" ixz="0"
-          iyy="0.033" iyz="0"
-          izz="0.00625"
+          ixx="0.1" ixy="0" ixz="0"
+          iyy="0.1" iyz="0"
+          izz="0.1"
       />
     </inertial>
@@ -84,7 +96,7 @@
       <origin xyz="0 0 0" rpy=" 0 1.5707 1.5707"/>
       <inertia
-          ixx="0.033" ixy="0" ixz="0"
-          iyy="0.033" iyz="0"
-          izz="0.00625"
+          ixx="0.1" ixy="0" ixz="0"
+          iyy="0.1" iyz="0"
+          izz="0.1"
       />
     </inertial>
@@ -150,5 +162,5 @@
   </link>
     <joint type="continuous" name="left_wheel_hinge">
-        <origin xyz="0 0.6 0" rpy="0 0 0"/>
+        <origin xyz="0 0.5 -0.125" rpy="0 0 0"/>
         <child link="left_wheel"/>
         <parent link="chassis"/>
@@ -158,13 +170,13 @@
     </joint>
     <joint type="continuous" name="right_wheel_hinge">
-        <origin xyz="0 -1 0" rpy="0 0 0"/>
+        <origin xyz="0 -0.5 -0.125" rpy="0 0 0"/>
         <child link="right_wheel"/>
         <parent link="chassis"/>
-        <axis xyz="0 -0.6 0" rpy="0 0 0"/>
+        <axis xyz="0 -1 0" rpy="0 0 0"/>
         <limit effort="10000" velocity="1000"/>
         <dynamics damping="1.0" friction="1.0"/>
     </joint>
     <joint type="fixed" name="camera_joint">
-        <origin xyz="0.5 0 0.1" rpy="0 0 0"/>
+        <origin xyz="0.5 0 0" rpy="0 0 0"/>
         <child link="camera"/>
         <parent link="chassis"/>
@@ -172,5 +184,5 @@
     </joint>
     <joint type="fixed" name="hokuyo_joint">
-        <origin xyz="0 0 1.2" rpy="0 0 0"/>
+        <origin xyz="0 0 1.5" rpy="0 0 0"/>
         <child link="hokuyo"/>
         <parent link="chassis"/>

Commit message: robot issue fixed

File: my_robot/urdf/my_robot.xacro (robot description, xacro)
@@ -44,5 +44,5 @@
     </visual>
     <collision name='back_caster_collision'>
-      <origin xyz="0.35 0 -0.22" rpy=" 0 0 0"/>
+      <origin xyz="0.35 0 -0.23" rpy=" 0 0 0"/>
       <geometry>
         <sphere radius="0.15"/>
@@ -50,5 +50,5 @@
     </collision>
     <visual name='back_caster_visual'>
-      <origin xyz="0.35 0 -0.22" rpy=" 0 0 0"/>
+      <origin xyz="0.35 0 -0.23" rpy=" 0 0 0"/>
       <geometry>
         <sphere radius="0.15"/>
@@ -56,5 +56,5 @@
     </visual>
     <collision name='front_caster_collision'>
-      <origin xyz="-0.35 0 -0.22" rpy=" 0 0 0"/>
+      <origin xyz="-0.35 0 -0.23" rpy=" 0 0 0"/>
       <geometry>
         <sphere radius="0.15"/>
@@ -62,5 +62,5 @@
     </collision>
     <visual name='front_caster_visual'>
-      <origin xyz="-0.35 0 -0.22" rpy=" 0 0 0"/>
+      <origin xyz="-0.35 0 -0.23" rpy=" 0 0 0"/>
       <geometry>
         <sphere radius="0.15"/>
@@ -102,5 +102,5 @@
     </inertial>
     <collision>
-      <origin xyz="0 0 0" rpy=" 0 1.5707 1.5707"/>
+      <origin xyz="0 0.1 0" rpy=" 0 1.5707 1.5707"/>
       <geometry>
         <cylinder radius=".25" length=".1"/>
@@ -151,5 +151,5 @@
       <origin xyz="0 0 0" rpy=" 0 0 0"/>
       <geometry>
-        <box size="0.1 0.1 0.1"/>
+        <box size="0.5 0.5 0.5"/>
       </geometry>
     </collision>
@@ -157,5 +157,5 @@
       <origin xyz="0 0 0" rpy=" 0 0 0"/>
       <geometry>
-      <mesh filename="file:///home/workspace/EllaCM/catkin_ws/src/my_robot/meshes/hokuyo.dae"/>
+        <mesh filename="file:///home/workspace/EllaCM/catkin_ws/src/UdacityProject2ROS/my_robot/meshes/hokuyo.dae"/>
       </geometry>
      </visual>
@@ -184,5 +184,5 @@
     </joint>
     <joint type="fixed" name="hokuyo_joint">
-        <origin xyz="0 0 1.5" rpy="0 0 0"/>
+        <origin xyz="0 0 0.8" rpy="0 0 0"/>
         <child link="hokuyo"/>
         <parent link="chassis"/>

Commit message: robot can move now! but it cannot go linearly bc of diff. in collision of its two wheels

File: my_robot/urdf/my_robot.xacro (robot description, xacro)
@@ -44,25 +44,25 @@
     </visual>
     <collision name='back_caster_collision'>
-      <origin xyz="0.35 0 -0.23" rpy=" 0 0 0"/>
+      <origin xyz="0.35 0 -0.19" rpy=" 0 0 0"/>
       <geometry>
-        <sphere radius="0.15"/>
+        <sphere radius="0.189"/>
       </geometry>
     </collision>
     <visual name='back_caster_visual'>
-      <origin xyz="0.35 0 -0.23" rpy=" 0 0 0"/>
+      <origin xyz="0.35 0 -0.19" rpy=" 0 0 0"/>
       <geometry>
-        <sphere radius="0.15"/>
+        <sphere radius="0.19"/>
       </geometry>
     </visual>
     <collision name='front_caster_collision'>
-      <origin xyz="-0.35 0 -0.23" rpy=" 0 0 0"/>
+      <origin xyz="-0.35 0 -0.19" rpy=" 0 0 0"/>
       <geometry>
-        <sphere radius="0.15"/>
+        <sphere radius="0.189"/>
       </geometry>
     </collision>
     <visual name='front_caster_visual'>
-      <origin xyz="-0.35 0 -0.23" rpy=" 0 0 0"/>
+      <origin xyz="-0.35 0 -0.19" rpy=" 0 0 0"/>
       <geometry>
-        <sphere radius="0.15"/>
+        <sphere radius="0.19"/>
       </geometry>
     </visual>
@@ -79,5 +79,5 @@
     </inertial>
     <collision>
-      <origin xyz="0 0 0" rpy=" 0 1.5707 1.5707"/>
+      <origin xyz="0 0.01 0.05" rpy=" 0 1.5707 1.5707"/>
       <geometry>
         <cylinder radius=".25" length=".1"/>
@@ -102,5 +102,5 @@
     </inertial>
     <collision>
-      <origin xyz="0 0.1 0" rpy=" 0 1.5707 1.5707"/>
+      <origin xyz="0 0 0.01" rpy=" 0 1.5707 1.5707"/>
       <geometry>
         <cylinder radius=".25" length=".1"/>
@@ -162,5 +162,5 @@
   </link>
     <joint type="continuous" name="left_wheel_hinge">
-        <origin xyz="0 0.5 -0.125" rpy="0 0 0"/>
+        <origin xyz="0 0.6 -0.125" rpy="0 0 0"/>
         <child link="left_wheel"/>
         <parent link="chassis"/>
@@ -170,5 +170,5 @@
     </joint>
     <joint type="continuous" name="right_wheel_hinge">
-        <origin xyz="0 -0.5 -0.125" rpy="0 0 0"/>
+        <origin xyz="0 -0.6 -0.125" rpy="0 0 0"/>
         <child link="right_wheel"/>
         <parent link="chassis"/>

Commit message: robot not tiled, but floating

File: my_robot/urdf/my_robot.xacro (robot description, xacro)
@@ -9,5 +9,5 @@
   </joint>
   <link name='chassis'>
-    <pose>0 0 -0.1 0 0 0</pose>
+    <pose>0 0 0 0 0 0</pose>
     <inertial>
       <mass value="20.0"/>
@@ -26,5 +26,5 @@
     </collision>
     <visual name='chassis_visual'>
-      <origin xyz="0 0 -0.1" rpy=" 0 0 0"/>
+      <origin xyz="0 0 0" rpy=" 0 0 0"/>
       <geometry>
         <cylinder radius=".5" length=".2"/>
@@ -32,37 +32,37 @@
     </visual>
     <collision name='body_tower'>
-      <origin xyz="0 0 0.3" rpy=" 0 0 0"/>
+      <origin xyz="0 0 -0.0" rpy=" 0 0 0"/>
       <geometry>
-        <box size="0.5 0.5 1"/>
+        <box size="0.5 0.5 0.8"/>
       </geometry>
     </collision>
     <visual name='body_tower'>
-      <origin xyz="0 0 0.3" rpy=" 0 0 0"/>
+      <origin xyz="0 0 0.35" rpy=" 0 0 0"/>
       <geometry>
-        <box size="0.5 0.5 1"/>
+        <box size="0.5 0.5 0.8"/>
       </geometry>
     </visual>
     <collision name='back_caster_collision'>
-      <origin xyz="0.35 0 -0.19" rpy=" 0 0 0"/>
+      <origin xyz="0.35 0 -0.065" rpy=" 0 0 0"/>
       <geometry>
-        <sphere radius="0.189"/>
+        <sphere radius="0.184"/>
       </geometry>
     </collision>
     <visual name='back_caster_visual'>
-      <origin xyz="0.35 0 -0.19" rpy=" 0 0 0"/>
+      <origin xyz="0.35 0 -0.065" rpy=" 0 0 0"/>
       <geometry>
-        <sphere radius="0.19"/>
+        <sphere radius="0.185"/>
       </geometry>
     </visual>
     <collision name='front_caster_collision'>
-      <origin xyz="-0.35 0 -0.19" rpy=" 0 0 0"/>
+      <origin xyz="-0.35 0 -0.065" rpy=" 0 0 0"/>
       <geometry>
-        <sphere radius="0.189"/>
+        <sphere radius="0.184"/>
       </geometry>
     </collision>
     <visual name='front_caster_visual'>
-      <origin xyz="-0.35 0 -0.19" rpy=" 0 0 0"/>
+      <origin xyz="-0.35 0 -0.065" rpy=" 0 0 0"/>
       <geometry>
-        <sphere radius="0.19"/>
+        <sphere radius="0.185"/>
       </geometry>
     </visual>
@@ -71,5 +71,5 @@
     <inertial>
       <mass value="5.0"/>
-      <origin xyz="0 0 0" rpy=" 0 0 0"/>
+      <origin xyz="0 0 0" rpy=" 0 1.5707 1.5707"/>
       <inertia
           ixx="0.1" ixy="0" ixz="0"
@@ -79,5 +79,5 @@
     </inertial>
     <collision>
-      <origin xyz="0 0.01 0.05" rpy=" 0 1.5707 1.5707"/>
+      <origin xyz="0 0 0" rpy=" 0 1.5707 1.5707"/>
       <geometry>
         <cylinder radius=".25" length=".1"/>
@@ -102,5 +102,5 @@
     </inertial>
     <collision>
-      <origin xyz="0 0 0.01" rpy=" 0 1.5707 1.5707"/>
+      <origin xyz="0 0 0" rpy=" 0 -1.5707 -1.5707"/>
       <geometry>
         <cylinder radius=".25" length=".1"/>
@@ -162,5 +162,5 @@
   </link>
     <joint type="continuous" name="left_wheel_hinge">
-        <origin xyz="0 0.6 -0.125" rpy="0 0 0"/>
+        <origin xyz="0 0.6 0" rpy="0 0 0"/>
         <child link="left_wheel"/>
         <parent link="chassis"/>
@@ -170,5 +170,5 @@
     </joint>
     <joint type="continuous" name="right_wheel_hinge">
-        <origin xyz="0 -0.6 -0.125" rpy="0 0 0"/>
+        <origin xyz="0 -0.6 0" rpy="0 0 0"/>
         <child link="right_wheel"/>
         <parent link="chassis"/>
@@ -178,5 +178,5 @@
     </joint>
     <joint type="fixed" name="camera_joint">
-        <origin xyz="0.5 0 0" rpy="0 0 0"/>
+        <origin xyz="0.49 0 0.1" rpy="0 0 0"/>
         <child link="camera"/>
         <parent link="chassis"/>

Commit message: robot looks like standing on the ground, but spins when driving it in straight line

File: my_robot/urdf/my_robot.xacro (robot description, xacro)
@@ -32,5 +32,5 @@
     </visual>
     <collision name='body_tower'>
-      <origin xyz="0 0 -0.0" rpy=" 0 0 0"/>
+      <origin xyz="0 0 0.35" rpy=" 0 0 0"/>
       <geometry>
         <box size="0.5 0.5 0.8"/>
@@ -44,5 +44,5 @@
     </visual>
     <collision name='back_caster_collision'>
-      <origin xyz="0.35 0 -0.065" rpy=" 0 0 0"/>
+      <origin xyz="0.35 0 -0.31" rpy=" 0 0 0"/>
       <geometry>
         <sphere radius="0.184"/>
@@ -50,5 +50,5 @@
     </collision>
     <visual name='back_caster_visual'>
-      <origin xyz="0.35 0 -0.065" rpy=" 0 0 0"/>
+      <origin xyz="0.35 0 -0.31" rpy=" 0 0 0"/>
       <geometry>
         <sphere radius="0.185"/>
@@ -56,5 +56,5 @@
     </visual>
     <collision name='front_caster_collision'>
-      <origin xyz="-0.35 0 -0.065" rpy=" 0 0 0"/>
+      <origin xyz="-0.35 0 -0.31" rpy=" 0 0 0"/>
       <geometry>
         <sphere radius="0.184"/>
@@ -62,5 +62,5 @@
     </collision>
     <visual name='front_caster_visual'>
-      <origin xyz="-0.35 0 -0.065" rpy=" 0 0 0"/>
+      <origin xyz="-0.35 0 -0.31" rpy=" 0 0 0"/>
       <geometry>
         <sphere radius="0.185"/>
@@ -162,5 +162,5 @@
   </link>
     <joint type="continuous" name="left_wheel_hinge">
-        <origin xyz="0 0.6 0" rpy="0 0 0"/>
+        <origin xyz="0 0.6 -0.25" rpy="0 0 0"/>
         <child link="left_wheel"/>
         <parent link="chassis"/>
@@ -170,5 +170,5 @@
     </joint>
     <joint type="continuous" name="right_wheel_hinge">
-        <origin xyz="0 -0.6 0" rpy="0 0 0"/>
+        <origin xyz="0 -0.6 -0.25" rpy="0 0 0"/>
         <child link="right_wheel"/>
         <parent link="chassis"/>

Commit message: pass the driving test!

File: my_robot/urdf/my_robot.xacro (robot description, xacro)
@@ -44,5 +44,5 @@
     </visual>
     <collision name='back_caster_collision'>
-      <origin xyz="0.35 0 -0.31" rpy=" 0 0 0"/>
+      <origin xyz="0.35 0 -0.06" rpy=" 0 0 0"/>
       <geometry>
         <sphere radius="0.184"/>
@@ -50,5 +50,5 @@
     </collision>
     <visual name='back_caster_visual'>
-      <origin xyz="0.35 0 -0.31" rpy=" 0 0 0"/>
+      <origin xyz="0.35 0 -0.06" rpy=" 0 0 0"/>
       <geometry>
         <sphere radius="0.185"/>
@@ -56,5 +56,5 @@
     </visual>
     <collision name='front_caster_collision'>
-      <origin xyz="-0.35 0 -0.31" rpy=" 0 0 0"/>
+      <origin xyz="-0.35 0 -0.06" rpy=" 0 0 0"/>
       <geometry>
         <sphere radius="0.184"/>
@@ -62,5 +62,5 @@
     </collision>
     <visual name='front_caster_visual'>
-      <origin xyz="-0.35 0 -0.31" rpy=" 0 0 0"/>
+      <origin xyz="-0.35 0 -0.06" rpy=" 0 0 0"/>
       <geometry>
         <sphere radius="0.185"/>
@@ -102,5 +102,5 @@
     </inertial>
     <collision>
-      <origin xyz="0 0 0" rpy=" 0 -1.5707 -1.5707"/>
+      <origin xyz="0 0 0" rpy=" 0 1.5707 1.5707"/>
       <geometry>
         <cylinder radius=".25" length=".1"/>
@@ -162,5 +162,5 @@
   </link>
     <joint type="continuous" name="left_wheel_hinge">
-        <origin xyz="0 0.6 -0.25" rpy="0 0 0"/>
+        <origin xyz="0 0.6 0.0" rpy="0 0 0"/>
         <child link="left_wheel"/>
         <parent link="chassis"/>
@@ -170,8 +170,8 @@
     </joint>
     <joint type="continuous" name="right_wheel_hinge">
-        <origin xyz="0 -0.6 -0.25" rpy="0 0 0"/>
+        <origin xyz="0 -0.6 0.0" rpy="0 0 0"/>
         <child link="right_wheel"/>
         <parent link="chassis"/>
-        <axis xyz="0 -1 0" rpy="0 0 0"/>
+        <axis xyz="0 1 0" rpy="0 0 0"/>
         <limit effort="10000" velocity="1000"/>
         <dynamics damping="1.0" friction="1.0"/>
